File: Ribv6.kicad_pcb (KiCad board)
At the start: 2 copper layers, 112 x 139 mm, 95 parts, among them J1 Conn_01x03, J10 Conn_01x19, J11 Conn_01x01_Male, J12 Conn_01x01_Male, J13 Conn_01x19, J14 Conn_02x07_Odd_Even, J15 Conn_02x07_Odd_Even, J16 Conn_01x19, J17 Conn_02x07_Odd_Even, J18 Conn_02x07_Odd_Even, J19 Conn_01x19, J2 Conn_01x03, J20 Conn_01x19, J21 Conn_01x19, J22 Conn_01x06, J23 Conn_02x06_Odd_Even, J24 Conn_01x01_Male, J25 Conn_01x06, J26 Conn_01x01_Male, J3 Conn_01x19, J4 Conn_02x07_Odd_Even, J5 Conn_01x19, J6 Conn_01x03, J7 Conn_01x19, J8 Conn_02x07_Odd_Even, J9 Conn_01x03, Q1 Q_PMOS_GDS, Q10 BSS138, Q11 BSS138, Q12 BSS138, Q13 BSS138, Q14 BSS138, Q15 BSS138, Q2 BSS138, Q3 BSS138, Q4 BSS138, Q5 BSS138, Q6 BSS138, Q7 Q_PMOS_GDS, Q8 BSS138, Q9 BSS138, U1 polulu-3784-D36V28F7, U2 polulu-3784-D36V28F7, U3 esp-devkit

Commit message: routing draft
Parts:
- J14, J15, J17, J18: value Conn_02x07_Odd_Even -> Conn_02x04_Odd_Even; footprint Connector_PinSocket_2.54mm:PinSocket_2x07_P2.54mm_Vertical -> Connector_PinSocket_2.54mm:PinSocket_2x04_P2.54mm_Vertical
- moved J10 250.6 mm to (6.95, -53.4)
- moved J7 245.7 mm to (9.49, -53.3)
- moved J9 238.2 mm to (12.0, -77.5), turned to 0 degrees
- moved J8 234.5 mm to (1.85, -68.6)
- moved F2 232.4 mm to (10.8, -58.9), turned to 180 degrees
- moved F3 223.4 mm to (7.01, -83.6), turned to 90 degrees
- moved J6 215.2 mm to (31.1, -77.5), turned to 0 degrees
- moved R22 200.2 mm to (41.7, -31.1)
- moved R23 200.2 mm to (41.7, -27.5)
- moved Q8 200.2 mm to (39.2, -30.8)
- moved Q9 200.2 mm to (39.2, -27.3)
- moved R17 200.2 mm to (36.6, -31.1)
- moved R18 200.2 mm to (36.6, -27.5)
- moved J21 197.8 mm to (57.7, -53.3)
- moved J24 193.3 mm to (69.6, -100.0)
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Connections:
- J16 pad 1: Net-(J13-Pad1) -> Net-(J16-Pad1)
- J16 pad 19: Net-(J13-Pad19) -> Net-(J16-Pad19)
- J19 pad 7: Net-(J19-Pad7) -> GND
- J20 pad 7: Net-(J20-Pad7) -> GND
- J21 pad 7: Net-(J21-Pad7) -> GND
- J22 pad 1: GPIO19_5 -> GPIO14_5
- J22 pad 2: GPIO18_5 -> GPIO25_5
- J22 pad 3: GPIO17_5 -> GPIO18_5
- J22 pad 5: GPIO25_5 -> GPIO19_5
- J22 pad 6: GPIO14_5 -> GPIO17_5
- U3 pad 3V3: Net-(J13-Pad1) -> +3.3VA
- U3 pad 5V: Net-(J13-Pad19) -> Net-(U3-Pad5V)
Routing:
- net +3V3: track 108.4 -> 325.5 mm, vias 3 -> 12
- net SCL_33: track 84.9 -> 243.7 mm, vias 0 -> 3
- net SDA_33: track 78.4 -> 218.2 mm, vias 0 -> 1
- net +5V: track 94.9 -> 226.7 mm, vias 10 -> 12
- net SDA_5: track 0.00 -> 106.8 mm, vias 0 -> 1
- net +3.3VA: track 0.00 -> 98.3 mm, vias 0 -> 6
- net SCL_5: track 0.00 -> 84.4 mm, vias 0 -> 1
- net GPIO17_5: track 0.00 -> 79.7 mm, vias 0 -> 1
- net GPIO19_5: track 0.00 -> 75.0 mm, vias 0 -> 1
- net GPIO16_5: track 0.00 -> 69.8 mm, vias 0 -> 1
- net Net-(F3-Pad1): track 58.4 -> 124.6 mm
- net GPIO18_5: track 0.00 -> 64.9 mm, vias 0 -> 1
- net GPIO25_5: track 0.00 -> 60.4 mm, vias 0 -> 1
- net GPIO14_5: track 0.00 -> 54.5 mm, vias 0 -> 1
- net Net-(D9-Pad2): track 0.00 -> 45.8 mm, vias 0 -> 2
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Other:
- board size 112 x 139 mm -> 193.8 x 121.7 mm
- board text added: "RIB Rev6 Kalbi"

Commit message: layout done, partial silk
Parts:
- removed J17, J18: Conn_02x04_Odd_Even, Connector_PinSocket_2.54mm:PinSocket_2x04_P2.54mm_Vertical
- added R38: 10k, Resistor_SMD:R_0603_1608Metric, F.Cu at (49.4, -50.6)
- moved J22 73.8 mm to (14.5, -5.08)
- moved J23 73.8 mm to (17.1, 7.62)
- moved R27 29.1 mm to (33.2, -24.6)
- moved R30 29.1 mm to (38.2, -24.6)
- moved Q13 29.1 mm to (35.7, -24.4)
- moved J14 23.4 mm to (70.4, 7.62), turned to 270 degrees
- moved R18 21.4 mm to (49.9, -44.3), turned to 90 degrees
- moved R29 21.3 mm to (49.9, -26.2), turned to 90 degrees
- moved Q9 19.1 mm to (47.3, -44.5), turned to 90 degrees
- moved R20 18.3 mm to (49.9, -33.7), turned to 90 degrees
- moved Q15 18.1 mm to (47.4, -26.5), turned to 90 degrees
- moved Q14 18.1 mm to (35.7, -32.0)
- moved R28 18.1 mm to (33.1, -32.2)
- moved R31 18.1 mm to (38.2, -32.2)
- moved R23 17.0 mm to (44.8, -44.3), turned to 270 degrees
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Connections:
- J13 pad 14: Net-(J13-Pad14) -> GND
- J13 pad 19: Net-(J13-Pad19) -> +5V
- J14 pad 2: +3V3 -> GND
- J14 pad 3: GND -> +3V3
- J14 pad 5: GND -> SCL_33
- J14 pad 6: +3V3 -> SCL_33
- J14 pad 7: GND -> SDA_33
- J14 pad 8: +3V3 -> SDA_33
- J15 pad 1: SDA_33 -> GND
- J15 pad 2: SCL_33 -> GND
- J15 pad 3: SDA_33 -> +5V
- J15 pad 4: SCL_33 -> +5V
- J15 pad 5: SDA_33 -> SCL_5
- J15 pad 6: SCL_33 -> SCL_5
- J15 pad 7: SDA_33 -> SDA_5
- J15 pad 8: SCL_33 -> SDA_5
- J16 pad 14: Net-(J13-Pad14) -> GND
- J16 pad 19: Net-(J16-Pad19) -> +5V
- J19 pad 11: Net-(J19-Pad11) -> GPIO17
- J20 pad 11: Net-(J19-Pad11) -> GPIO17
- J21 pad 11: Net-(J19-Pad11) -> GPIO17
- J22 pad 3: GPIO18_5 -> GPIO19_5
- J22 pad 4: GPIO16_5 -> GPIO18_5
- J22 pad 5: GPIO19_5 -> GPIO17_5
- J22 pad 6: GPIO17_5 -> GPIO16_5
- J25 pad 2: Net-(J25-Pad2) -> prez
- U3 pad 5V: Net-(U3-Pad5V) -> +5V
- U3 pad GND: Net-(J13-Pad14) -> GND
- U3 pad IO17: Net-(J19-Pad11) -> GPIO17
Routing:
- net +5V: track 226.7 -> 364.2 mm, vias 12 -> 27
- net SCL_33: track 243.7 -> 170.5 mm, vias 3 -> 2
- net prez: track 0.00 -> 60.8 mm, vias 0 -> 1
- net SDA_33: track 218.2 -> 165.2 mm, vias 1 -> 3
- net Net-(J3-Pad1): track 0.00 -> 45.7 mm
- net SDA_5: track 106.8 -> 63.2 mm, vias 1 -> 2
- net GPIO14: track 50.7 -> 15.1 mm
- net GPIO16: track 48.8 -> 17.1 mm, vias 4 -> 0
- net GPIO19: track 43.8 -> 17.4 mm, vias 1 -> 0
- net GPIO25: track 41.3 -> 15.1 mm, vias 2 -> 0
- net GPIO18: track 41.9 -> 18.0 mm, vias 2 -> 0
- net GPIO17_5: track 79.7 -> 59.6 mm, vias 1 -> 0
- net GPIO17: track 1.60 -> 17.4 mm
- net UBEC2: track 68.6 -> 84.3 mm, vias 1 -> 3
- net SCL_5: track 84.4 -> 70.5 mm, vias 1 -> 2
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- added copper zone on In1.Cu, net GND
- added copper zone on In2.Cu, net GND
Other:
- board size 193.8 x 121.7 mm -> 85 x 116.3 mm
- copper layers 2 -> 4

Commit message: re-laying out power section.
Parts:
- added U4: DPDT_x2, GF-126-0327:GF-126-0327, F.Cu at (102.1, 65.3)
- R1, R16, R33, R35, R36, R37: value R_Small -> 330
- moved J1 232.5 mm to (247.8, 18.8)
- moved Q4 232.5 mm to (276.8, 18.9)
- moved Q5 232.5 mm to (264.6, 18.9)
- moved Q6 232.5 mm to (268.7, 18.9)
- moved R10 232.5 mm to (264.9, 22.9)
- moved R11 232.5 mm to (264.9, 21.4)
- moved R2 232.5 mm to (260.8, 22.9)
- moved R3 232.5 mm to (260.8, 21.4)
- moved R4 232.5 mm to (273.0, 22.9)
- moved R5 232.5 mm to (273.0, 21.4)
- moved J2 232.5 mm to (228.7, 18.8)
- moved J6 232.5 mm to (242.8, 18.8)
- moved J9 232.5 mm to (223.6, 18.8)
- moved Q2 232.5 mm to (260.5, 18.9)
- moved Q3 232.5 mm to (272.7, 18.9)
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Connections:
- F3 pad 2: +BATT -> Net-(F3-Pad2)
- J3 pad 1: Net-(J3-Pad1) -> GND
- J3 pad 10: Net-(J3-Pad1) -> GND
- J3 pad 11: Net-(J3-Pad1) -> GND
- J3 pad 12: Net-(J3-Pad1) -> GND
- J3 pad 13: Net-(J3-Pad1) -> GND
- J3 pad 14: Net-(J3-Pad1) -> GND
- J3 pad 15: Net-(J3-Pad1) -> GND
- J3 pad 16: Net-(J3-Pad1) -> GND
- J3 pad 17: Net-(J3-Pad1) -> GND
- J3 pad 18: Net-(J3-Pad1) -> GND
- J3 pad 19: Net-(J3-Pad1) -> GND
- J3 pad 2: Net-(J3-Pad1) -> GND
- J3 pad 3: Net-(J3-Pad1) -> GND
- J3 pad 4: Net-(J3-Pad1) -> GND
- J3 pad 5: Net-(J3-Pad1) -> GND
- J3 pad 6: Net-(J3-Pad1) -> GND
- J3 pad 7: Net-(J3-Pad1) -> GND
- J3 pad 8: Net-(J3-Pad1) -> GND
- J3 pad 9: Net-(J3-Pad1) -> GND
Routing:
- net +3V3: track 333.5 -> 249.7 mm, vias 22 -> 15
- net Net-(F3-Pad1): track 124.6 -> 62.4 mm
- net Net-(J3-Pad1): track 45.7 -> 0.00 mm
- net GND: track 30.2 -> 75.9 mm
- net Net-(F3-Pad2): track 0.00 -> 29.4 mm
- net UBEC2: track 84.3 -> 59.1 mm
- net prez: track 60.8 -> 71.2 mm
- net SDA_33: track 165.2 -> 175.2 mm
- net SCL_33: track 170.5 -> 179.0 mm
- net +BATT: track 179.7 -> 172.0 mm
- net GPIO16_5: track 60.1 -> 53.1 mm
- net GPIO17_5: track 59.6 -> 53.1 mm
- net GPIO18_5: track 62.7 -> 56.3 mm
- net GPIO25_5: track 52.4 -> 46.3 mm
- net GPIO19_5: track 62.0 -> 55.9 mm
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Other:
- board size 85 x 116.3 mm -> 84.7 x 126.2 mm
- board text added: "3"
- board text added: "3v"
- board text added: "3v Fuse"
- board text added: "3v Reg"
- board text added: "5"
- board text added: "5V IO"
- board text added: "5v"
- board text added: "5v Fuse"
- board text added: "5v Reg"
- board text added: "B"
- board text added: "B E C"
- board text added: "BAT"
- board text added: "BEC1"
- board text added: "BEC2"
- board text added: "C"
- board text added: "CLK"
- board text added: "CMD"
- board text added: "D"
- board text added: "EN"
- board text added: "G"
- board text added: "GND"
- board text added: "IIC 3V"
- board text added: "IIC 5V"
- board text added: "IO1"
- board text added: "IO12"
- board text added: "IO13"
- board text added: "IO14"
- board text added: "IO15"
- board text added: "IO16"
- board text added: "IO17"
- board text added: "IO18"
- board text added: "IO19"
- board text added: "IO2"
- board text added: "IO21"
- board text added: "IO22"
- board text added: "IO23"
- board text added: "IO25"
- board text added: "IO26"
- board text added: "IO27"
- board text added: "IO32"
- board text added: "IO33"
- board text added: "IO34"
- board text added: "IO35"
- board text added: "IO4"
- board text added: "IO5"
- board text added: "L Bank Fuse"
- board text added: "L Bank Pow"
- board text added: "Main Fuse"
- board text added: "R Bank Fuse"
- board text added: "R Bank Pow"
- board text added: "RX0"
- board text added: "SD0"
- board text added: "SD1"
- board text added: "SD2"
- board text added: "SD3"
- board text added: "SVN"
- board text added: "SVP"
- board text added: "TX0"
- board text added: "U"
