File: _autosave-Ribv6.kicad_pcb (KiCad board)
At the start: 4 copper layers, 84.7 x 126.2 mm, 93 parts, among them J1 Conn_01x03, J10 Conn_01x19, J11 Conn_01x01_Male, J12 Conn_01x01_Male, J13 Conn_01x19, J14 Conn_02x04_Odd_Even, J15 Conn_02x04_Odd_Even, J16 Conn_01x19, J19 Conn_01x19, J2 Conn_01x02_Female, J20 Conn_01x19, J21 Conn_01x19, J22 Conn_01x06, J23 Conn_02x06_Odd_Even, J24 Conn_01x01_Male, J25 Conn_01x06, J26 Conn_01x01_Male, J3 Conn_01x19, J4 Conn_02x07_Odd_Even, J5 Conn_01x19, J6 Conn_01x02_Female, J7 Conn_01x19, J8 Conn_02x07_Odd_Even, J9 Conn_01x03, Q1 BSS138, Q10 BSS138, Q11 BSS138, Q12 BSS138, Q13 BSS138, Q14 BSS138, Q15 BSS138, Q2 BSS138, Q3 BSS138, Q4 BSS138, Q5 BSS138, Q6 BSS138, Q7 BSS138, Q8 BSS138, Q9 BSS138, U1 polulu-3784-D36V28F7, U2 polulu-3784-D36V28F7, U3 esp-devkit, U4 DPDT_x2

Commit message: more routing
Routing:
- net Net-(D7-Pad1): track 0.00 -> 53.1 mm, vias 0 -> 1
- net GND: track 61.8 -> 66.8 mm
- net UBEC1: track 9.53 -> 13.1 mm
- net Net-(Q6-Pad1): track 0.00 -> 3.24 mm
Changed lines of the file:
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@@
     (thickness 1.6)
     (drawings 100)
-    (tracks 705)
+    (tracks 727)
     (zones 0)
     (modules 93)
@@
   (segment (start 154.8069 60.6204) (end 154.3796 60.6204) (width 0.25) (layer F.Cu) (net 1))
   (segment (start 154.3796 60.6204) (end 153.25 61.75) (width 0.25) (layer F.Cu) (net 1))
+  (segment (start 133.6071 88.1674) (end 133.5156 88.2589) (width 0.25) (layer F.Cu) (net 1))
+  (segment (start 135.0556 88.1674) (end 133.6071 88.1674) (width 0.25) (layer F.Cu) (net 1))
+  (segment (start 133.4656 88.2589) (end 133.5156 88.2589) (width 0.25) (layer F.Cu) (net 1))
+  (segment (start 132.588 87.3813) (end 133.4656 88.2589) (width 0.25) (layer F.Cu) (net 1))
+  (segment (start 132.588 85.217) (end 132.588 87.3813) (width 0.25) (layer F.Cu) (net 1))
   (segment (start 162.5625 94.15) (end 162.4625 94.25) (width 0.25) (layer F.Cu) (net 2))
   (segment (start 162.5625 92.25) (end 162.5625 94.15) (width 0.25) (layer F.Cu) (net 2))
@@
   (segment (start 136.5 76.5) (end 133.899999 79.100001) (width 0.25) (layer F.Cu) (net 7))
   (segment (start 119.899999 79.100001) (end 133.899999 79.100001) (width 0.25) (layer F.Cu) (net 7))
+  (segment (start 131.5156 88.5589) (end 130.5 87.5433) (width 0.25) (layer F.Cu) (net 9))
+  (segment (start 131.5156 89.2089) (end 131.5156 88.5589) (width 0.25) (layer F.Cu) (net 9))
+  (segment (start 130.5 87.5433) (end 130.5 84.75) (width 0.25) (layer F.Cu) (net 9))
+  (via (at 134.25 82.75) (size 0.8) (drill 0.4) (layers F.Cu B.Cu) (net 9))
+  (segment (start 130.5 84.75) (end 132.5 82.75) (width 0.25) (layer F.Cu) (net 9))
+  (segment (start 132.5 82.75) (end 134.25 82.75) (width 0.25) (layer F.Cu) (net 9))
+  (segment (start 134.25 82.75) (end 137.5 82.75) (width 0.25) (layer B.Cu) (net 9))
+  (segment (start 158.599001 86.138001) (end 160.75 83.987002) (width 0.25) (layer B.Cu) (net 9))
+  (segment (start 137.5 82.75) (end 140.888001 86.138001) (width 0.25) (layer B.Cu) (net 9))
+  (segment (start 140.888001 86.138001) (end 158.599001 86.138001) (width 0.25) (layer B.Cu) (net 9))
+  (segment (start 160.75 83.987002) (end 160.75 70.769176) (width 0.25) (layer B.Cu) (net 9))
+  (segment (start 160.75 70.769176) (end 159.604494 69.62367) (width 0.25) (layer B.Cu) (net 9))
   (segment (start 158.035 84.963) (end 142.795 84.963) (width 2) (layer F.Cu) (net 10))
   (segment (start 143.125 92.505) (end 143.125 89.105) (width 2) (layer F.Cu) (net 10))
@@
   (segment (start 140.445 82.423) (end 139.451001 83.416999) (width 1.5) (layer F.Cu) (net 15))
   (segment (start 142.795 82.423) (end 140.445 82.423) (width 1.5) (layer F.Cu) (net 15))
+  (segment (start 136.5796 86.6686) (end 135.128 85.217) (width 0.25) (layer F.Cu) (net 15))
+  (segment (start 136.5796 88.1674) (end 136.5796 86.6686) (width 0.25) (layer F.Cu) (net 15))
   (segment (start 120.785899 143.234419) (end 123.04522 145.49374) (width 1.5) (layer B.Cu) (net 16))
   (segment (start 123.04522 145.49374) (end 129.24282 151.69134) (width 1.5) (layer B.Cu) (net 16))
@@
   (segment (start 114.837 89.7875) (end 114.4656 90.1589) (width 0.25) (layer F.Cu) (net 62))
   (segment (start 116 89.7875) (end 114.837 89.7875) (width 0.25) (layer F.Cu) (net 62))
+  (segment (start 136.5796 89.7424) (end 135.0556 89.7424) (width 0.25) (layer F.Cu) (net 64))
+  (segment (start 134.6391 90.1589) (end 135.0556 89.7424) (width 0.25) (layer F.Cu) (net 64))
+  (segment (start 133.5156 90.1589) (end 134.6391 90.1589) (width 0.25) (layer F.Cu) (net 64))
   (segment (start 148.4503 114.0841) (end 135.7503 114.0841) (width 0.25) (layer F.Cu) (net 65))
   (segment (start 131.4388 113.2028) (end 131.3973 113.1613) (width 0.25) (layer F.Cu) (net 65))
